File: flatbox-halal-low-prof/flatbox-halal-low-prof.kicad_sch (KiCad schematic)
At the start: 21 parts, among them SW1 SW_Push, SW10 SW_Push, SW11 SW_Push, SW12 SW_Push, SW13 SW_Push, SW14 SW_Push, SW15 SW_Push, SW16 SW_Push, SW17 SW_Push, SW18 SW_Push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

Commit message: cleaned up signal trace
Parts:
- added H1, H2, H3, H4: MountingHole, MountingHole:MountingHole_6.4mm_M6, symbol Mechanical:MountingHole
