File: halalsnackbox-kicad/halalsnackbox.kicad_sch (KiCad schematic)
At the start: 25 parts, among them SW1 SW_Push, SW10 SW_Push, SW11 SW_Push, SW12 SW_Push, SW13 SW_Push, SW14 SW_Push, SW15 SW_Push, SW16 SW_Push, SW17 SW_Push, SW18 SW_Push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

Commit message: Modified file structure
Parts:
- A1: footprint RP2040-Zero:RP2040-Zero -> halalsnackbox-footprints:RP2040-Zero
- H1, H2, H3, H4: footprint MountingHole:MountingHole_6.4mm_M6 -> halalsnackbox-footprints:MountingHole_6.4mm_M6
- SW1, SW2, SW3, SW4, SW5, SW6: footprint Button_Switch_THT:SW_PUSH_6mm_H5mm -> halalsnackbox-footprints:SW_PUSH_6mm
- SW10, SW11, SW12, SW13, SW14, SW15, SW16, SW17, SW18, SW19, SW20, SW7, SW8, SW9: footprint key-switches:SW_Gateron_LowProfile_HotSwap_THT -> halalsnackbox-footprints:SW_Gateron_LowProfile_HotSwap_THT

Commit message: Added freecad file for 3d printed case
Parts:
- H1, H2, H3, H4: footprint halalsnackbox-footprints:MountingHole_6.4mm_M6 -> MountingHole:MountingHole_6.4mm_M6
- SW1, SW2, SW3, SW4, SW5, SW6: footprint halalsnackbox-footprints:SW_PUSH_6mm -> halalsnackbox-footprints:SW_PUSH_6mm_H9.5mm
Changed lines of the file:
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@@
 			)
 		)
-		(property "Footprint" "halalsnackbox-footprints:SW_PUSH_6mm"
+		(property "Footprint" "halalsnackbox-footprints:SW_PUSH_6mm_H9.5mm"
 			(at 45.72 60.96 0)
 			(effects
@@
 			)
 		)
-		(property "Footprint" "halalsnackbox-footprints:SW_PUSH_6mm"
+		(property "Footprint" "halalsnackbox-footprints:SW_PUSH_6mm_H9.5mm"
 			(at 63.5 60.96 0)
 			(effects
@@
 			)
 		)
-		(property "Footprint" "halalsnackbox-footprints:SW_PUSH_6mm"
+		(property "Footprint" "halalsnackbox-footprints:SW_PUSH_6mm_H9.5mm"
 			(at 81.28 60.96 0)
 			(effects
@@
 			)
 		)
-		(property "Footprint" "halalsnackbox-footprints:SW_PUSH_6mm"
+		(property "Footprint" "halalsnackbox-footprints:SW_PUSH_6mm_H9.5mm"
 			(at 99.06 60.96 0)
 			(effects
@@
 			)
 		)
-		(property "Footprint" "halalsnackbox-footprints:SW_PUSH_6mm"
+		(property "Footprint" "halalsnackbox-footprints:SW_PUSH_6mm_H9.5mm"
 			(at 116.84 60.96 0)
 			(effects
@@
 			)
 		)
-		(property "Footprint" "halalsnackbox-footprints:SW_PUSH_6mm"
+		(property "Footprint" "halalsnackbox-footprints:SW_PUSH_6mm_H9.5mm"
 			(at 134.62 60.96 0)
 			(effects
@@
 			)
 		)
-		(property "Footprint" "halalsnackbox-footprints:MountingHole_6.4mm_M6"
+		(property "Footprint" "MountingHole:MountingHole_6.4mm_M6"
 			(at 162.56 123.19 0)
 			(effects
@@
 			)
 		)
-		(property "Footprint" "halalsnackbox-footprints:MountingHole_6.4mm_M6"
+		(property "Footprint" "MountingHole:MountingHole_6.4mm_M6"
 			(at 162.56 128.27 0)
 			(effects
@@
 			)
 		)
-		(property "Footprint" "halalsnackbox-footprints:MountingHole_6.4mm_M6"
+		(property "Footprint" "MountingHole:MountingHole_6.4mm_M6"
 			(at 162.56 118.11 0)
 			(effects
@@
 			)
 		)
-		(property "Footprint" "halalsnackbox-footprints:MountingHole_6.4mm_M6"
+		(property "Footprint" "MountingHole:MountingHole_6.4mm_M6"
 			(at 162.56 133.35 0)
 			(effects
